Commit message: adding variables with xacro

File: src/rip_description/urdf/rotary_pend.urdf.xacro (robot description, xacro)
@@ -1,3 +1,7 @@
-<robot name="rotary_inverted_pendulum">
+<?xml version="1.0"?>
+<robot name="rotary_inverted_pendulum" xmlns:xacro="http://www.ros.org/wiki/xacro">
+    <xacro:property name = "base_height" value="0.3" />
+    <xacro:property name = "arm_length" value="0.06 " />
+    <xacro:property name = "pendulum_length" value="0.2 " />
     <material name="grey">
         <color rgba="0.7 0.7 0.7 1"/>
@@ -12,7 +16,7 @@
         <visual>
             <geometry>
-                <cylinder radius="0.05" length="0.3"/>
+                <cylinder radius="0.05" length="${base_height}"/>
             </geometry>
-            <origin xyz="0 0 0.15" rpy="0 0 0"/>
+            <origin xyz="0 0 ${base_height / 2}" rpy="0 0 0"/>
             <material name="green"/>
         </visual>
@@ -21,7 +25,7 @@
         <visual>
             <geometry>
-                <box size="0.06 0.03 0.01"/>
+                <box size="${arm_length} 0.03 0.01"/>
             </geometry>
-            <origin xyz="0.03 0 0" rpy="0 0 0"/>
+            <origin xyz="${arm_length / 2} 0 0" rpy="0 0 0"/>
             <material name="grey"/>
         </visual>
@@ -30,7 +34,7 @@
         <visual>
             <geometry>
-                <box size="0.2 0.03 0.01"/>
+                <box size="${pendulum_length} 0.03 0.01"/>
             </geometry>
-            <origin xyz="0.1  0 0" rpy="0 0 0"/>
+            <origin xyz="${pendulum_length / 2}  0 0" rpy="0 0 0"/>
             <material name="red"/>
         </visual>
@@ -39,14 +43,14 @@
         <parent link="base_link"/>
         <child link="arm_link"/>
-        <origin xyz="0 0 0.30" rpy="0 0 0"/>
+        <origin xyz="0 0 ${base_height}" rpy="0 0 0"/>
         <axis xyz="0 0 1"/>
-        <limit effort="10" lower="-3.1416" upper="3.1416" velocity="1.0"/>
+        <limit effort="10" lower="-${pi}" upper="${pi}" velocity="1.0"/>
     </joint>
     <joint name="arm_pendulum_joint" type="revolute">
         <parent link="arm_link"/>
         <child link="pendulum_link"/>
-        <origin xyz="0.06 0 0" rpy="0 1.5708 0"/>
+        <origin xyz="${arm_length} 0 0" rpy="0 ${pi / 2.0} 0"/>
         <axis xyz="0 0 1"/>
-        <limit effort="10" lower="-3.1416" upper="3.1416" velocity="1.0"/>
+        <limit effort="10" lower="-${pi}" upper="${pi}" velocity="1.0"/>
     </joint>
 </robot>
